Commit message: Activacion control JoinStatus de rviz con vision artificial

File: install/roshandia_pkg/share/roshandia_pkg/urdf/hand.urdf (robot description, URDF)
Before this commit: robot handIA, 8 links, 7 joints
Joints:
- joint f1_to_hand: axis 0.707 0 0.707 -> 0.707 0.707 0.707

Commit message: gazebo

File: install/roshandia_pkg/share/roshandia_pkg/urdf/hand.urdf (robot description, URDF)
Before this commit: robot handIA, 8 links, 7 joints
Links:
- link arm: mass None -> 0.5
- link blade: mass None -> 0.5
- link finger1: mass None -> 0.5
- link finger2: mass None -> 0.5
- link finger3: mass None -> 0.5
- link finger4: mass None -> 0.5
- link finger5: mass None -> 0.5
- link hand: mass None -> 0.5
Joints:
- joint f1_to_hand: limit lower=-1 upper=1 effort=100 velocity=0.5 -> lower=-1 upper=1 effort=100 velocity=2
- joint f2_to_hand: limit lower=-1.222 upper=0 effort=100 velocity=0.5 -> lower=-1.222 upper=0 effort=100 velocity=2
- joint f3_to_hand: limit lower=-1.222 upper=0 effort=100 velocity=0.5 -> lower=-1.222 upper=0 effort=100 velocity=2
